Commit message: lidar and rgbd camera mocks

File: ros2_ws/src/rover_description/urdf/rover.urdf.xacro (robot description, xacro)
@@ -4,4 +4,17 @@
   <xacro:arg name="robot_ns" default=""/>
   <xacro:arg name="mecanum_wheels" default="false"/>
+  <xacro:arg name="lidar_xyz" default="0.1 0 0.15"/>
+  <xacro:arg name="lidar_rpy" default="0 0 0"/>
+  <xacro:arg name="depth_camera_xyz" default="0.1746 0 0.0906"/>
+  <xacro:arg name="depth_camera_rpy" default="0 0.4712 0"/>
+  <xacro:property name="robot_ns_arg" value="$(arg robot_ns)"/>
+  <xacro:property name="link_prefix" value=""/>
+  <xacro:property name="joint_prefix" value=""/>
+  <xacro:property name="topic_prefix" value=""/>
+  <xacro:if value="${robot_ns_arg != '' and robot_ns_arg != '/'}">
+    <xacro:property name="link_prefix" value="${robot_ns_arg}/"/>
+    <xacro:property name="joint_prefix" value="${robot_ns_arg}_"/>
+    <xacro:property name="topic_prefix" value="${robot_ns_arg}/"/>
+  </xacro:if>
   <xacro:include filename="$(find leo_description)/urdf/macros.xacro"/>
   <xacro:leo_sim robot_ns="$(arg robot_ns)"
@@ -18,5 +31,5 @@
     </plugin>
   </gazebo>
-  <link name="lidar_link">
+  <link name="${link_prefix}lidar_link">
     <visual>
       <geometry>
@@ -28,8 +41,73 @@
     </visual>
   </link>
-  <joint name="lidar_joint" type="fixed">
-    <parent link="base_link"/>
-    <child link="lidar_link"/>
-    <origin xyz="0.1 0 0.15" rpy="0 0 0"/>
+  <link name="${link_prefix}depth_camera_link">
+    <visual>
+      <geometry>
+        <mesh filename="package://rover_description/meshes/camera.stl" scale="0.001 0.001 0.001"/>
+      </geometry>
+    </visual>
+  </link>
+  <link name="${link_prefix}depth_camera_optical_frame"/>
+  <joint name="${joint_prefix}lidar_joint" type="fixed">
+    <parent link="${link_prefix}base_link"/>
+    <child link="${link_prefix}lidar_link"/>
+    <origin xyz="$(arg lidar_xyz)" rpy="$(arg lidar_rpy)"/>
   </joint>
+  <joint name="${joint_prefix}depth_camera_joint" type="fixed">
+    <parent link="${link_prefix}base_link"/>
+    <child link="${link_prefix}depth_camera_link"/>
+    <origin xyz="$(arg depth_camera_xyz)" rpy="$(arg depth_camera_rpy)"/>
+  </joint>
+  <joint name="${joint_prefix}depth_camera_optical_joint" type="fixed">
+    <parent link="${link_prefix}depth_camera_link"/>
+    <child link="${link_prefix}depth_camera_optical_frame"/>
+    <origin xyz="0 0 0" rpy="-1.57079632679 0 -1.57079632679"/>
+  </joint>
+  <gazebo reference="${link_prefix}lidar_link">
+    <sensor name="lidar_sensor" type="gpu_lidar">
+      <always_on>true</always_on>
+      <update_rate>10</update_rate>
+      <visualize>true</visualize>
+      <topic>${topic_prefix}scan</topic>
+      <gz_frame_id>${link_prefix}lidar_link</gz_frame_id>
+      <lidar>
+        <scan>
+          <horizontal>
+            <samples>720</samples>
+            <resolution>1</resolution>
+            <min_angle>-3.14159</min_angle>
+            <max_angle>3.14159</max_angle>
+          </horizontal>
+        </scan>
+        <range>
+          <min>0.15</min>
+          <max>12.0</max>
+          <resolution>0.01</resolution>
+        </range>
+      </lidar>
+    </sensor>
+  </gazebo>
+  <gazebo reference="${link_prefix}depth_camera_link">
+    <sensor name="depth_camera_sensor" type="rgbd_camera">
+      <always_on>1</always_on>
+      <update_rate>10</update_rate>
+      <visualize>true</visualize>
+      <topic>${topic_prefix}depth_camera</topic>
+      <gz_frame_id>${link_prefix}depth_camera_optical_frame</gz_frame_id>
+      <camera name="depth_camera">
+        <camera_info_topic>${topic_prefix}depth_camera/camera_info</camera_info_topic>
+        <horizontal_fov>1.047</horizontal_fov>
+        <image>
+          <width>320</width>
+          <height>240</height>
+          <format>R8G8B8</format>
+        </image>
+        <clip>
+          <near>0.05</near>
+          <far>5.0</far>
+        </clip>
+        <optical_frame_id>${link_prefix}depth_camera_optical_frame</optical_frame_id>
+      </camera>
+    </sensor>
+  </gazebo>
 </robot>

Commit message: Add proper camera and lidar to model

File: ros2_ws/src/rover_description/urdf/rover.urdf.xacro (robot description, xacro)
@@ -4,5 +4,5 @@
   <xacro:arg name="robot_ns" default=""/>
   <xacro:arg name="mecanum_wheels" default="false"/>
-  <xacro:arg name="lidar_xyz" default="0.1 0 0.15"/>
+  <xacro:arg name="lidar_xyz" default="0.0700 0 0.0380"/>
   <xacro:arg name="lidar_rpy" default="0 0 0"/>
   <xacro:arg name="depth_camera_xyz" default="0.1746 0 0.0906"/>
@@ -34,9 +34,6 @@
     <visual>
       <geometry>
-        <cylinder radius="0.05" length="0.05"/>
+        <mesh filename="package://rover_description/meshes/lidar.stl" scale="0.001 0.001 0.001"/>
       </geometry>
-      <material name="black">
-        <color rgba="0 0 0 1"/>
-      </material>
     </visual>
   </link>
